File: RelayBoard/RelayBoard.kicad_pcb (KiCad board)
At the start: 2 copper layers, 203.2 x 94 mm, 23 parts, among them J1 Conn_Coaxial, J2 Conn_Coaxial, J3 Conn_01x06_Female, K1 G5LE-1, K2 G5LE-1, K3 G5LE-1, K4 G5LE-1, K5 G5LE-1, K6 G5LE-1, K7 G5LE-1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

Commit message: layout the relay borad
Parts:
- removed the Q3 at (156.2, 142.9)
- added Q4: 2SC1815, Package_TO_SOT_THT:TO-92_Inline_Wide, F.Cu at (217.2, 140.3)
- Q1, Q2: footprint Package_TO_SOT_THT:TO-92_Inline -> Package_TO_SOT_THT:TO-92_Inline_Wide
- Q3: renamed from Q4; footprint Package_TO_SOT_THT:TO-92_Inline -> Package_TO_SOT_THT:TO-92_Inline_Wide
- R1, R2, R3, R4: footprint Resistor_SMD:R_0603_1608Metric_Pad1.05x0.95mm_HandSolder -> Resistor_SMD:R_0805_2012Metric_Pad1.15x1.40mm_HandSolder
- moved J3 104.2 mm to (130.8, 139.7)
- moved Q3 38.8 mm to (166.4, 140.3), turned to 180 degrees
- moved D1 32.8 mm to (58.9, 112.3), turned to 0 degrees
- moved D2 30.7 mm to (105.2, 112.3)
- moved D3 29.8 mm to (156.0, 112.3)
- moved D4 29.6 mm to (206.8, 112.3)
- moved R2 8.74 mm to (115.2, 140.3), turned to 0 degrees
- moved R1 8.59 mm to (65.0, 140.3), turned to 0 degrees
- moved R4 4.94 mm to (207.3, 140.3), turned to 180 degrees
- moved Q2 4.58 mm to (103.5, 140.3), turned to 0 degrees
- moved Q1 4.07 mm to (54.6, 140.3), turned to 0 degrees
- moved K8 3.70 mm to (211.5, 116.8)
- moved R3 3.59 mm to (155.8, 140.3), turned to 180 degrees
- moved K4 3.42 mm to (211.5, 72.4)
- moved J1 3.17 mm to (53.3, 84.5)
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Connections:
- J3 pad 1: +12V -> GND
- J3 pad 2: sw0 -> sw1
- J3 pad 3: sw1 -> sw0
- J3 pad 4: sw2 -> sw3
- J3 pad 5: sw3 -> sw2
- J3 pad 6: GND -> +12V
- K1 pad 4: Net-(K1-Pad4) -> Net-(K1-Pad3)
- K2 pad 2: Net-(D3-Pad2) -> Net-(D2-Pad2)
- K2 pad 4: Net-(K2-Pad4) -> Net-(K2-Pad3)
- K3 pad 2: Net-(D4-Pad2) -> Net-(D3-Pad2)
- K3 pad 4: Net-(K3-Pad4) -> Net-(K3-Pad3)
- K4 pad 2: Net-(D2-Pad2) -> Net-(D4-Pad2)
- K4 pad 4: Net-(K4-Pad4) -> Net-(K4-Pad3)
- K5 pad 4: Net-(K5-Pad4) -> Net-(K5-Pad3)
- K6 pad 4: Net-(K6-Pad4) -> Net-(K6-Pad3)
- K6 pad 5: Net-(D3-Pad2) -> Net-(D2-Pad2)
- K7 pad 4: Net-(K7-Pad4) -> Net-(K7-Pad3)
- K7 pad 5: Net-(D4-Pad2) -> Net-(D3-Pad2)
- K8 pad 4: Net-(K8-Pad4) -> Net-(K8-Pad3)
- K8 pad 5: Net-(D2-Pad2) -> Net-(D4-Pad2)
- Q3 pad 2: Net-(D4-Pad2) -> Net-(D3-Pad2)
- Q3 pad 3: Net-(Q4-Pad3) -> Net-(Q3-Pad3)
- R2 pad 2: sw3 -> sw1
- R3 pad 2: sw1 -> sw2
- R4 pad 2: sw2 -> sw3
Routing:
- net +12V: track 197.6 -> 458.4 mm
- net sw0: track 0.00 -> 73.5 mm
- net sw3: track 0.00 -> 72.2 mm
- net Net-(J2-Pad1): track 184.7 -> 229.0 mm
- net Net-(D1-Pad2): track 49.5 -> 77.3 mm
- net Net-(D2-Pad2): track 49.1 -> 74.8 mm
- net Net-(D3-Pad2): track 49.1 -> 73.0 mm
- net Net-(D4-Pad2): track 49.1 -> 72.0 mm
- net sw1: track 0.00 -> 21.2 mm
- net sw2: track 0.00 -> 15.6 mm
- net Net-(J1-Pad1): track 210.1 -> 223.8 mm
- net Net-(Q2-Pad3): track 0.00 -> 5.57 mm
- net Net-(Q3-Pad3): track 0.00 -> 4.44 mm
- net Net-(Q1-Pad3): track 0.00 -> 4.30 mm
- net Net-(Q4-Pad3): track 0.00 -> 3.81 mm
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- added copper zone on B.Cu, net GND
- added copper zone on F.Cu, net GND
- added copper zone on F.Cu, net Net-(J1-Pad1)

Commit message: add another trial amp,
Parts:
- K1, K2, K3, K4, K5, K6, K7, K8: footprint Relay_THT:Relay_SPDT_Omron-G5LE-1 -> Myfootprint:Relay_SPST_Omron-G5LE
Routing:
- net Net-(K5-Pad3): track 0.00 -> 17.1 mm
- net +12V: track 458.4 -> 457.3 mm
- net Net-(D3-Pad2): track 73.0 -> 72.4 mm
- net Net-(D1-Pad2): track 77.3 -> 76.7 mm
- net sw2: track 15.6 -> 16.1 mm
Other:
- board size 203.2 x 94 mm -> 203.7 x 94 mm
