File: RelayBoard/RelayBoard.sch (KiCad schematic (older format))
At the start: 23 parts, among them J1 Conn_Coaxial, J2 Conn_Coaxial, J3 Conn_01x06_Female, K1 G5LE-1, K2 G5LE-1, K3 G5LE-1, K4 G5LE-1, K5 G5LE-1, K6 G5LE-1, K7 G5LE-1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

Commit message: layout the relay borad
Parts:
- Q1: footprint Package_TO_SOT_THT:TO-92_Inline -> Package_TO_SOT_THT:TO-92_Inline_Wide
- Q2: renamed from Q3; footprint Package_TO_SOT_THT:TO-92_Inline -> Package_TO_SOT_THT:TO-92_Inline_Wide
- Q3: renamed from Q4; footprint Package_TO_SOT_THT:TO-92_Inline -> Package_TO_SOT_THT:TO-92_Inline_Wide
- Q4: renamed from Q2; footprint Package_TO_SOT_THT:TO-92_Inline -> Package_TO_SOT_THT:TO-92_Inline_Wide
- R1: footprint Resistor_SMD:R_0603_1608Metric_Pad1.05x0.95mm_HandSolder -> Resistor_SMD:R_0805_2012Metric_Pad1.15x1.40mm_HandSolder
- R2: renamed from R3; footprint Resistor_SMD:R_0603_1608Metric_Pad1.05x0.95mm_HandSolder -> Resistor_SMD:R_0805_2012Metric_Pad1.15x1.40mm_HandSolder
- R3: renamed from R4; footprint Resistor_SMD:R_0603_1608Metric_Pad1.05x0.95mm_HandSolder -> Resistor_SMD:R_0805_2012Metric_Pad1.15x1.40mm_HandSolder
- R4: renamed from R2; footprint Resistor_SMD:R_0603_1608Metric_Pad1.05x0.95mm_HandSolder -> Resistor_SMD:R_0805_2012Metric_Pad1.15x1.40mm_HandSolder
- renumbered D3 to D2, D4 to D3, D2 to D4
Connections:
- net +12V: now also J3.6 (Pin_6); no longer J3.1 (Pin_1)
- net GND: now also J3.1 (Pin_1); no longer J3.6 (Pin_6)
- net sw0: now also J3.3 (Pin_3); no longer J3.2 (Pin_2)
- net sw1: now also J3.2 (Pin_2); no longer J3.3 (Pin_3)
- net sw2: now also J3.5 (Pin_5); no longer J3.4 (Pin_4)
- net sw3: now also J3.4 (Pin_4); no longer J3.5 (Pin_5)
- net at K1.3: now also K1.4
- net at K2.3: now also K2.4
- net at K3.3: now also K3.4
- net at K4.3: now also K4.4
- net at K5.3: now also K5.4
- net at K6.3: now also K6.4
- net at K7.3: now also K7.4
- net at K8.3: now also K8.4
Changed lines of the file:
@@
 F 0 "R1" V 1645 1750 50  0000 C CNN
 F 1 "2k" V 1736 1750 50  0000 C CNN
-F 2 "Resistor_SMD:R_0603_1608Metric_Pad1.05x0.95mm_HandSolder" V 1890 1740 50  0001 C CNN
+F 2 "Resistor_SMD:R_0805_2012Metric_Pad1.15x1.40mm_HandSolder" V 1890 1740 50  0001 C CNN
 F 3 "~" H 1850 1750 50  0001 C CNN
 	1    1850 1750
@@
 F 0 "Q1" H 2490 1796 50  0000 L CNN
 F 1 "2SC1815" H 2490 1705 50  0000 L CNN
-F 2 "Package_TO_SOT_THT:TO-92_Inline" H 2500 1675 50  0001 L CIN
+F 2 "Package_TO_SOT_THT:TO-92_Inline_Wide" H 2500 1675 50  0001 L CIN
 F 3 "https://media.digikey.com/pdf/Data%20Sheets/Toshiba%20PDFs/2SC1815.pdf" H 2300 1750 50  0001 L CNN
 	1    2300 1750
@@
 Connection ~ 2800 2900
 $Comp
-L Device:D D3
+L Device:D D2
 U 1 1 62E83480
 P 2800 2750
-F 0 "D3" V 2754 2829 50  0000 L CNN
+F 0 "D2" V 2754 2829 50  0000 L CNN
 F 1 "D" V 2845 2829 50  0000 L CNN
 F 2 "Diode_THT:D_T-1_P10.16mm_Horizontal" H 2800 2750 50  0001 C CNN
@@
 $EndComp
 $Comp
-L Device:R_US R3
+L Device:R_US R2
 U 1 1 62E8348C
 P 1900 3150
-F 0 "R3" V 1695 3150 50  0000 C CNN
+F 0 "R2" V 1695 3150 50  0000 C CNN
 F 1 "2k" V 1786 3150 50  0000 C CNN
-F 2 "Resistor_SMD:R_0603_1608Metric_Pad1.05x0.95mm_HandSolder" V 1940 3140 50  0001 C CNN
+F 2 "Resistor_SMD:R_0805_2012Metric_Pad1.15x1.40mm_HandSolder" V 1940 3140 50  0001 C CNN
 F 3 "~" H 1900 3150 50  0001 C CNN
 	1    1900 3150
@@
 $EndComp
 $Comp
-L Transistor_BJT:2SC1815 Q3
+L Transistor_BJT:2SC1815 Q2
 U 1 1 62E83492
 P 2350 3150
-F 0 "Q3" H 2540 3196 50  0000 L CNN
+F 0 "Q2" H 2540 3196 50  0000 L CNN
 F 1 "2SC1815" H 2540 3105 50  0000 L CNN
-F 2 "Package_TO_SOT_THT:TO-92_Inline" H 2550 3075 50  0001 L CIN
+F 2 "Package_TO_SOT_THT:TO-92_Inline_Wide" H 2550 3075 50  0001 L CIN
 F 3 "https://media.digikey.com/pdf/Data%20Sheets/Toshiba%20PDFs/2SC1815.pdf" H 2350 3150 50  0001 L CNN
 	1    2350 3150
@@
 Connection ~ 2850 4200
 $Comp
-L Device:D D4
+L Device:D D3
 U 1 1 62E85137
 P 2850 4050
-F 0 "D4" V 2804 4129 50  0000 L CNN
+F 0 "D3" V 2804 4129 50  0000 L CNN
 F 1 "D" V 2895 4129 50  0000 L CNN
 F 2 "Diode_THT:D_T-1_P10.16mm_Horizontal" H 2850 4050 50  0001 C CNN
@@
 $EndComp
 $Comp
-L Device:R_US R4
+L Device:R_US R3
 U 1 1 62E85143
 P 1950 4450
-F 0 "R4" V 1745 4450 50  0000 C CNN
+F 0 "R3" V 1745 4450 50  0000 C CNN
 F 1 "2k" V 1836 4450 50  0000 C CNN
-F 2 "Resistor_SMD:R_0603_1608Metric_Pad1.05x0.95mm_HandSolder" V 1990 4440 50  0001 C CNN
+F 2 "Resistor_SMD:R_0805_2012Metric_Pad1.15x1.40mm_HandSolder" V 1990 4440 50  0001 C CNN
 F 3 "~" H 1950 4450 50  0001 C CNN
 	1    1950 4450
@@
 $EndComp
 $Comp
-L Transistor_BJT:2SC1815 Q4
+L Transistor_BJT:2SC1815 Q3
 U 1 1 62E85149
 P 2400 4450
-F 0 "Q4" H 2590 4496 50  0000 L CNN
+F 0 "Q3" H 2590 4496 50  0000 L CNN
 F 1 "2SC1815" H 2590 4405 50  0000 L CNN
-F 2 "Package_TO_SOT_THT:TO-92_Inline" H 2600 4375 50  0001 L CIN
+F 2 "Package_TO_SOT_THT:TO-92_Inline_Wide" H 2600 4375 50  0001 L CIN
 F 3 "https://media.digikey.com/pdf/Data%20Sheets/Toshiba%20PDFs/2SC1815.pdf" H 2400 4450 50  0001 L CNN
 	1    2400 4450
@@
 Connection ~ 2750 5450
 $Comp
-L Device:D D2
+L Device:D D4
 U 1 1 62E87CC8
 P 2750 5300
-F 0 "D2" V 2704 5379 50  0000 L CNN
+F 0 "D4" V 2704 5379 50  0000 L CNN
 F 1 "D" V 2795 5379 50  0000 L CNN
 F 2 "Diode_THT:D_T-1_P10.16mm_Horizontal" H 2750 5300 50  0001 C CNN
@@
 $EndComp
 $Comp
-L Device:R_US R2
+L Device:R_US R4
 U 1 1 62E87CD4
 P 1850 5700
-F 0 "R2" V 1645 5700 50  0000 C CNN
+F 0 "R4" V 1645 5700 50  0000 C CNN
 F 1 "2k" V 1736 5700 50  0000 C CNN
-F 2 "Resistor_SMD:R_0603_1608Metric_Pad1.05x0.95mm_HandSolder" V 1890 5690 50  0001 C CNN
+F 2 "Resistor_SMD:R_0805_2012Metric_Pad1.15x1.40mm_HandSolder" V 1890 5690 50  0001 C CNN
 F 3 "~" H 1850 5700 50  0001 C CNN
 	1    1850 5700
@@
 $EndComp
 $Comp
-L Transistor_BJT:2SC1815 Q2
+L Transistor_BJT:2SC1815 Q4
 U 1 1 62E87CDA
 P 2300 5700
-F 0 "Q2" H 2490 5746 50  0000 L CNN
+F 0 "Q4" H 2490 5746 50  0000 L CNN
 F 1 "2SC1815" H 2490 5655 50  0000 L CNN
-F 2 "Package_TO_SOT_THT:TO-92_Inline" H 2500 5625 50  0001 L CIN
+F 2 "Package_TO_SOT_THT:TO-92_Inline_Wide" H 2500 5625 50  0001 L CIN
 F 3 "https://media.digikey.com/pdf/Data%20Sheets/Toshiba%20PDFs/2SC1815.pdf" H 2300 5700 50  0001 L CNN
 	1    2300 5700
@@
 L power:+12V #PWR012
 U 1 1 62EC1F12
-P 8350 950
-F 0 "#PWR012" H 8350 800 50  0001 C CNN
-F 1 "+12V" H 8365 1123 50  0000 C CNN
-F 2 "" H 8350 950 50  0001 C CNN
-F 3 "" H 8350 950 50  0001 C CNN
-	1    8350 950
-	1    0    0    -1
-$EndComp
-Wire Wire Line
-	8350 1050 8350 950
+P 7550 1550
+F 0 "#PWR012" H 7550 1400 50  0001 C CNN
+F 1 "+12V" H 7565 1723 50  0000 C CNN
+F 2 "" H 7550 1550 50  0001 C CNN
+F 3 "" H 7550 1550 50  0001 C CNN
+	1    7550 1550
+	1    0    0    -1
+$EndComp
 Wire Wire Line
 	8350 1150 8050 1150
@@
 L power:GND #PWR013
 U 1 1 62ECD8C3
-P 8350 1700
-F 0 "#PWR013" H 8350 1450 50  0001 C CNN
-F 1 "GND" H 8355 1527 50  0000 C CNN
-F 2 "" H 8350 1700 50  0001 C CNN
-F 3 "" H 8350 1700 50  0001 C CNN
-	1    8350 1700
-	1    0    0    -1
-$EndComp
-Wire Wire Line
-	8350 1700 8350 1550
+P 7550 1050
+F 0 "#PWR013" H 7550 800 50  0001 C CNN
+F 1 "GND" H 7555 877 50  0000 C CNN
+F 2 "" H 7550 1050 50  0001 C CNN
+F 3 "" H 7550 1050 50  0001 C CNN
+	1    7550 1050
+	1    0    0    -1
+$EndComp
+Text GLabel 8050 1250 0    50   Input ~ 0
+sw0
 Text GLabel 8050 1150 0    50   Input ~ 0
-sw0
-Text GLabel 8050 1250 0    50   Input ~ 0
 sw1
+Text GLabel 8050 1450 0    50   Input ~ 0
+sw2
 Text GLabel 8050 1350 0    50   Input ~ 0
-sw2
-Text GLabel 8050 1450 0    50   Input ~ 0
 sw3
 Text GLabel 1700 1750 0    50   Input ~ 0
@@
 Wire Wire Line
 	7650 5200 7650 6500
+Wire Wire Line
+	8350 1050 7550 1050
+Wire Wire Line
+	8350 1550 7550 1550
+Wire Wire Line
+	3550 2150 3550 1950
+Wire Wire Line
+	3600 3550 3600 3350
+Wire Wire Line
+	3650 4650 3650 4850
+Wire Wire Line
+	3550 6100 3550 5900
+Wire Wire Line
+	6000 6000 6000 6200
+Wire Wire Line
+	6000 4850 6000 4650
+Wire Wire Line
+	6000 3300 6000 3500
+Wire Wire Line
+	6000 1950 6000 2150
 $EndSCHEMATC

Commit message: add another trial amp,
Parts:
- K1, K2, K3, K4, K5, K6, K7, K8: footprint Relay_THT:Relay_SPDT_Omron-G5LE-1 -> Myfootprint:Relay_SPST_Omron-G5LE; symbol Relay:G5LE-1 -> Mylib:G5LE-1A_SPST
Changed lines of the file:
@@
 	1    0    0    -1
-$EndComp
-$Comp
-L Relay:G5LE-1 K1
-U 1 1 62E80542
-P 3250 1850
-F 0 "K1" V 2683 1850 50  0000 C CNN
-F 1 "G5LE-1" V 2774 1850 50  0000 C CNN
-F 2 "Relay_THT:Relay_SPDT_Omron-G5LE-1" H 3700 1800 50  0001 L CNN
-F 3 "http://www.omron.com/ecb/products/pdf/en-g5le.pdf" H 3250 1850 50  0001 C CNN
-	1    3250 1850
-	0    1    1    0
 $EndComp
 Wire Wire Line
@@
 $EndComp
 $Comp
-L Relay:G5LE-1 K2
+L Mylib:G5LE-1A_SPST K2
 U 1 1 62E83498
 P 3300 3250
 F 0 "K2" V 2733 3250 50  0000 C CNN
 F 1 "G5LE-1" V 2824 3250 50  0000 C CNN
-F 2 "Relay_THT:Relay_SPDT_Omron-G5LE-1" H 3750 3200 50  0001 L CNN
+F 2 "Myfootprint:Relay_SPST_Omron-G5LE" H 3750 3200 50  0001 L CNN
 F 3 "http://www.omron.com/ecb/products/pdf/en-g5le.pdf" H 3300 3250 50  0001 C CNN
 	1    3300 3250
@@
 $EndComp
 $Comp
-L Relay:G5LE-1 K3
+L Mylib:G5LE-1A_SPST K3
 U 1 1 62E8514F
 P 3350 4550
 F 0 "K3" V 2783 4550 50  0000 C CNN
 F 1 "G5LE-1" V 2874 4550 50  0000 C CNN
-F 2 "Relay_THT:Relay_SPDT_Omron-G5LE-1" H 3800 4500 50  0001 L CNN
+F 2 "Myfootprint:Relay_SPST_Omron-G5LE" H 3800 4500 50  0001 L CNN
 F 3 "http://www.omron.com/ecb/products/pdf/en-g5le.pdf" H 3350 4550 50  0001 C CNN
 	1    3350 4550
@@
 $EndComp
 $Comp
-L Relay:G5LE-1 K4
+L Mylib:G5LE-1A_SPST K4
 U 1 1 62E87CE0
 P 3250 5800
 F 0 "K4" V 2683 5800 50  0000 C CNN
 F 1 "G5LE-1" V 2774 5800 50  0000 C CNN
-F 2 "Relay_THT:Relay_SPDT_Omron-G5LE-1" H 3700 5750 50  0001 L CNN
+F 2 "Myfootprint:Relay_SPST_Omron-G5LE" H 3700 5750 50  0001 L CNN
 F 3 "http://www.omron.com/ecb/products/pdf/en-g5le.pdf" H 3250 5800 50  0001 C CNN
 	1    3250 5800
@@
 $EndComp
 $Comp
-L Relay:G5LE-1 K5
+L Mylib:G5LE-1A_SPST K5
 U 1 1 62E8C862
 P 5700 1850
 F 0 "K5" V 5133 1850 50  0000 C CNN
 F 1 "G5LE-1" V 5224 1850 50  0000 C CNN
-F 2 "Relay_THT:Relay_SPDT_Omron-G5LE-1" H 6150 1800 50  0001 L CNN
+F 2 "Myfootprint:Relay_SPST_Omron-G5LE" H 6150 1800 50  0001 L CNN
 F 3 "http://www.omron.com/ecb/products/pdf/en-g5le.pdf" H 5700 1850 50  0001 C CNN
 	1    5700 1850
@@
 $EndComp
 $Comp
-L Relay:G5LE-1 K6
+L Mylib:G5LE-1A_SPST K6
 U 1 1 62E930D5
 P 5700 3200
 F 0 "K6" V 5133 3200 50  0000 C CNN
 F 1 "G5LE-1" V 5224 3200 50  0000 C CNN
-F 2 "Relay_THT:Relay_SPDT_Omron-G5LE-1" H 6150 3150 50  0001 L CNN
+F 2 "Myfootprint:Relay_SPST_Omron-G5LE" H 6150 3150 50  0001 L CNN
 F 3 "http://www.omron.com/ecb/products/pdf/en-g5le.pdf" H 5700 3200 50  0001 C CNN
 	1    5700 3200
@@
 $EndComp
 $Comp
-L Relay:G5LE-1 K7
+L Mylib:G5LE-1A_SPST K7
 U 1 1 62E95284
 P 5700 4550
 F 0 "K7" V 5133 4550 50  0000 C CNN
 F 1 "G5LE-1" V 5224 4550 50  0000 C CNN
-F 2 "Relay_THT:Relay_SPDT_Omron-G5LE-1" H 6150 4500 50  0001 L CNN
+F 2 "Myfootprint:Relay_SPST_Omron-G5LE" H 6150 4500 50  0001 L CNN
 F 3 "http://www.omron.com/ecb/products/pdf/en-g5le.pdf" H 5700 4550 50  0001 C CNN
 	1    5700 4550
@@
 $EndComp
 $Comp
-L Relay:G5LE-1 K8
+L Mylib:G5LE-1A_SPST K8
 U 1 1 62E9789A
 P 5700 5900
 F 0 "K8" V 5133 5900 50  0000 C CNN
 F 1 "G5LE-1" V 5224 5900 50  0000 C CNN
-F 2 "Relay_THT:Relay_SPDT_Omron-G5LE-1" H 6150 5850 50  0001 L CNN
+F 2 "Myfootprint:Relay_SPST_Omron-G5LE" H 6150 5850 50  0001 L CNN
 F 3 "http://www.omron.com/ecb/products/pdf/en-g5le.pdf" H 5700 5900 50  0001 C CNN
 	1    5700 5900
@@
 	8350 1550 7550 1550
 Wire Wire Line
+	3600 3550 3600 3350
+Wire Wire Line
+	3650 4650 3650 4850
+Wire Wire Line
+	3550 6100 3550 5900
+Wire Wire Line
+	6000 6000 6000 6200
+Wire Wire Line
+	6000 4850 6000 4650
+Wire Wire Line
+	6000 3300 6000 3500
+Wire Wire Line
+	6000 1950 6000 2150
+Wire Wire Line
 	3550 2150 3550 1950
-Wire Wire Line
-	3600 3550 3600 3350
-Wire Wire Line
-	3650 4650 3650 4850
-Wire Wire Line
-	3550 6100 3550 5900
-Wire Wire Line
-	6000 6000 6000 6200
-Wire Wire Line
-	6000 4850 6000 4650
-Wire Wire Line
-	6000 3300 6000 3500
-Wire Wire Line
-	6000 1950 6000 2150
+$Comp
+L Mylib:G5LE-1A_SPST K1
+U 1 1 62E80542
+P 3250 1850
+F 0 "K1" V 2683 1850 50  0000 C CNN
+F 1 "G5LE-1" V 2774 1850 50  0000 C CNN
+F 2 "Myfootprint:Relay_SPST_Omron-G5LE" H 3700 1800 50  0001 L CNN
+F 3 "http://www.omron.com/ecb/products/pdf/en-g5le.pdf" H 3250 1850 50  0001 C CNN
+	1    3250 1850
+	0    1    1    0
+$EndComp
 $EndSCHEMATC
