File: PA/GeneralPA/GeneralPA.sch (KiCad schematic (older format))
At the start: 119 parts, among them J2 RFin, J3 RFout, J4 FAN, J5 SWR, J6 48v_PAD, J7 48v_PAD, Q1 2N3904, Q2 IRF510, Q3 IRF510, Q4 IRF510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

Commit message: update 2nd version of PA, adding some driver ciruits
Parts:
- removed L9: 33n, Myfootprint:HomeMade_L_aircore, symbol pspice:INDUCTOR
- removed Q4: IRF510, Package_TO_SOT_THT:TO-220-3_Horizontal_TabDown, symbol Transistor_FET:IRF540N
- removed TP2, TP3: Conn_Coaxial, Connector_Coaxial:U.FL_Molex_MCRF_73412-0110_Vertical, symbol Connector:Conn_Coaxial
- added C30: 10n, Capacitor_SMD:C_0805_2012Metric_Pad1.15x1.40mm_HandSolder, symbol Device:C_Small
- added C35: 10u, Capacitor_SMD:C_1206_3216Metric_Pad1.42x1.75mm_HandSolder, symbol Device:C_Small
- added C44: 100n, Capacitor_SMD:C_0805_2012Metric_Pad1.15x1.40mm_HandSolder, symbol Device:C_Small
- added C45: 0.1u, Capacitor_SMD:C_0805_2012Metric_Pad1.15x1.40mm_HandSolder, symbol Device:C_Small
- added C46: 150p, Capacitor_SMD:C_1206_3216Metric_Pad1.42x1.75mm_HandSolder, symbol Device:C_Small
- added J1: FAN, Connector_PinHeader_2.54mm:PinHeader_1x02_P2.54mm_Vertical, symbol Connector:Conn_01x02_Male
- added Q4: 2sc5706, Package_TO_SOT_SMD:TO-252-2, symbol Transistor_BJT:2SD1047
- added R1: 390, Resistor_SMD:R_0805_2012Metric_Pad1.15x1.40mm_HandSolder, symbol Device:R_Small_US
- added R23: 270/0.25W, Resistor_THT:R_Axial_DIN0411_L9.9mm_D3.6mm_P12.70mm_Horizontal, symbol Device:R_Small_US
- added R24: 22/1W, Resistor_THT:R_Axial_DIN0411_L9.9mm_D3.6mm_P12.70mm_Horizontal, symbol Device:R_Small_US
- added R25: 3.3/0.5W, Resistor_THT:R_Axial_DIN0411_L9.9mm_D3.6mm_P12.70mm_Horizontal, symbol Device:R_Small_US
- added R26: 0, Resistor_SMD:R_0815_2038Metric_Pad1.53x4.00mm_HandSolder, symbol Device:R_Small_US
- added RV3, RV4: 1k, Potentiometer_THT:Potentiometer_Bourns_3266Y_Vertical, symbol Device:R_POT_US
- added T4: Transformer_1P_1S, GeneralPA:HomeMade_Transformer_T50, symbol Device:Transformer_1P_1S
- C17: value 0.1u -> 10u; footprint Capacitor_SMD:C_0805_2012Metric_Pad1.15x1.40mm_HandSolder -> Capacitor_SMD:C_1206_3216Metric_Pad1.42x1.75mm_HandSolder
- C2, C8: value 1n -> 100n
- C26: value 0.1u -> 100n
- C32: renamed from C?; value 4.7n -> 100n
- H10, H4, H5, H6, H7, H8, H9: footprint Myfootprint:T50_Laminent -> GeneralPA:T50_Laminent
- J2, J3: footprint Connector_Coaxial:SMA_Amphenol_132289_EdgeMount -> Connector_Coaxial:SMA_Molex_73251-1153_EdgeMount_Horizontal
- L1, L2, L3, L4, L7, L8: footprint Myfootprint:HomeMade_L_aircore -> GeneralPA:HomeMade_L_aircore
- L12, L13: footprint Myfootprint:HomeMade_T50_1t33t -> GeneralPA:HomeMade_T50_1t33t
- L5: footprint Inductor_THT:L_Axial_L14.0mm_D4.5mm_P7.62mm_Vertical_Fastron_LACC -> Inductor_THT:L_Axial_L7.0mm_D3.3mm_P5.08mm_Vertical_Fastron_MICC
- L6: footprint Myfootprint:HomeMade_BalChoke -> GeneralPA:HomeMade_BalChoke
- Q1, Q6: footprint Package_TO_SOT_THT:TO-92_Inline -> Package_TO_SOT_THT:TO-92_Inline_Wide
- Q5: footprint Package_TO_SOT_THT:TO-251-2-1EP_Horizontal_TabDown -> Package_TO_SOT_SMD:TO-252-2; symbol Transistor_BJT:2SC1945 -> Transistor_BJT:2SD1047
- R12: value 680 -> 3.3
- R13: value 620 -> 1k
- R16: value 330 -> 470
- R21: value 7.1/1W -> 51; footprint Resistor_THT:R_Axial_DIN0411_L9.9mm_D3.6mm_P12.70mm_Horizontal -> Resistor_SMD:R_0805_2012Metric_Pad1.15x1.40mm_HandSolder
- R22: value 560/1W -> 270; footprint Resistor_THT:R_Axial_DIN0411_L9.9mm_D3.6mm_P12.70mm_Horizontal -> Resistor_SMD:R_0805_2012Metric_Pad1.15x1.40mm_HandSolder
- R4: value 200 -> 100
- R5: value 120 -> 100
- R6: value 5.1 -> 3.3
- T1, T2: footprint Myfootprint:HomeMade_Transformer_T50 -> GeneralPA:HomeMade_Transformer_T50
- T3: footprint Myfootprint:HomeMade_Transformer_T100 -> GeneralPA:HomeMade_Transformer_T100
- U2: value LM7809_TO220 -> LM7812_TO220
- gave numbers to parts that had none: 1
Connections:
- net GND: now also C26.2, R16.2, C30.2, J1.1 (Pin_1), R1.2, R24.2, R25.2, RV3.3, RV4.3; no longer C17.2, C32.2, R13.2, T1.2 (AB)
- net vshut: now also R29.1, R30.2, U1.1 (ADJ); no longer C17.1, R12.1, R16.2
- net at C8.1, Q5.1 (B), R10.2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: now also R1.1, RV3.2; no longer R13.1
- net at C32.1, R21.1: now also Q5.3 (E); no longer Q5.2 (E)
- net at C21.1: now also T4.1 (AA), T4.3 (SA); no longer L5.2
- net at R22.2: now also C17.2; no longer C21.2
- net +24V: now reaches C26.1
- net +24V: now also C37.1, J4.2 (Pin_2), L14.2, L5.1, R13.1, R29.2, T1.2 (AB), U1.2 (VO), C30.1, J1.2 (Pin_2)
- net at C24.1, R2.1, T1.1 (AA): no longer TP1.1 (In)
- net at R2.2: now also C45.1, R26.2; no longer C26.2
- net at C25.2, L7.2, T3.4 (SB): now also C46.2
- net at C25.1, L8.2, T3.3 (SA): now also C46.1
- removed net +28V: C16.1, C18.1, C37.1, J4.2 (Pin_2), L14.2, L5.1, R29.2, U1.2 (VO)
- net +9V renamed +12V
- net +12V: now also C16.1, C18.1, T4.2 (AB); no longer R16.1
- new net: C17.1, Q5.2 (C), T4.4 (SB)
- new net: C21.2, Q4.1 (B), R13.2, R16.1, R23.1, RV4.2
- new net: C32.2, R12.1
- new net: C44.2, R25.1
- new net: C44.1, Q4.3 (E), R24.1
- new net: C35.2, R23.2
- new net: C35.1, L5.2, Q4.2 (C), R26.1
- new net: C45.2, TP1.1 (In)
Other:
- note added: "0.1A for 0.5W output"
- note added: "DNS"
- moved on the sheet: C16, C17, C18, C21, J4, J6, J7, R22, TP1
